Commit message: update robot urdf file,add base_footprint and small pillar

File: ROSCode/src/description/urdf/robot.urdf (robot description, URDF)
Before this commit: robot my_robot, 32 links, 31 joints
Links:
- added link arduino_board; visual box size=0.11 0.06 0.005
- added link base_footprint; visual box size=0.005 0.005 0.005
- added link battery; visual box size=0.15 0.135 0.04
- added link left_blue_A_pillar; visual box size=0.04 0.01 0.003
- added link left_blue_B_pillar; visual box size=0.045 0.01 0.003
- added link left_blue_pillar; visual box size=0.025 0.025 0.002
- added link pi_board; visual box size=0.075 0.095 0.005
- added link right_blue_A_pillar; visual box size=0.04 0.01 0.003
- added link right_blue_B_pillar; visual box size=0.045 0.01 0.003
- added link right_blue_pillar; visual box size=0.025 0.025 0.002
- link A_motor: geometry visual cylinder length=0.12 radius=0.015
- link A_wheel: geometry visual cylinder length=0.025 radius=0.029
- link B_motor: geometry visual cylinder length=0.12 radius=0.015
- link B_wheel: geometry visual cylinder length=0.025 radius=0.029
- link C_motor: geometry visual cylinder length=0.12 radius=0.015
- link C_wheel: geometry visual cylinder length=0.025 radius=0.029
Joints:
- added joint base_footprint_joint: type fixed, parent base_footprint, child base_link, origin xyz=0 0 0.058
- added joint base_to_arduino: type fixed, parent base_link, child arduino_board, origin xyz=0 0 0.005
- added joint battery_joint: type fixed, parent B_pannel, child battery, origin xyz=0 0 0.022
- added joint left_blue_A_joint: type fixed, parent left_blue_pillar, child left_blue_A_pillar, origin xyz=0.017 0.013 -0.003 rpy=0 0 0.611
- added joint left_blue_B_joint: type fixed, parent left_blue_A_pillar, child left_blue_B_pillar, origin xyz=0.032 -0.015 0.0 rpy=0 0 -0.851
- added joint left_blue_pillar_joint: type fixed, parent blue_C_pillar, child left_blue_pillar, origin xyz=0 0.0165 0.025
- added joint pi_board_joint: type fixed, parent Pi_pannel, child pi_board, origin xyz=-0.06 0 0.005
- added joint right_blue_A_joint: type fixed, parent right_blue_pillar, child right_blue_A_pillar, origin xyz=0.017 -0.013 -0.003 rpy=0 0 -0.611
- added joint right_blue_B_joint: type fixed, parent right_blue_A_pillar, child right_blue_B_pillar, origin xyz=0.032 0.015 0.0 rpy=0 0 0.851
- added joint right_blue_pillar_joint: type fixed, parent blue_C_pillar, child right_blue_pillar, origin xyz=0 -0.0165 0.025
- joint base_to_A_wheel: origin xyz=0.09 -0.1559 -0.035 rpy=1.57079 0 0.5236 -> xyz=0.08725 -0.1511 -0.029 rpy=1.57079 0 0.5236
- joint base_to_B_wheel: origin xyz=0.09 0.1559 -0.035 rpy=1.57075 0 -0.5236 -> xyz=0.08725 0.1511 -0.029 rpy=1.57075 0 -0.5236
- joint base_to_C_wheel: origin xyz=-0.17 0 -0.035 rpy=1.57075 0 1.57 -> xyz=-0.1745 0 -0.029 rpy=1.57075 0 1.57

Commit message: update robot urdf and amcl code

File: ROSCode/src/description/urdf/robot.urdf (robot description, URDF)
Before this commit: robot my_robot, 42 links, 41 joints
Links:
- removed link IMU_sensor
- removed link lidar
- added link base_imu_link; visual box size=0.025 0.018 0.002
- added link laser; visual cylinder length=0.042 radius=0.038
Joints:
- joint lidar_to_pannel: child lidar -> laser
- joint pi_pannel_to_IMU: child IMU_sensor -> base_imu_link
